Commit message: Created a yaml file and modified the urdf

File: nuturtle_description/urdf/turtlebot3_burger.urdf.xacro (robot description, xacro)
@@ -2,5 +2,11 @@
 <robot name="turtlebot3_burger"
   xmlns:xacro="http://ros.org/wiki/xacro">
-  <!-- <xacro:include filename="$(find turtlebot3_description)/urdf/common_properties.urdf"/> -->
+<xacro:property name="yaml_file" value="$(find nuturtle_description)/config/diff_params.yaml"/>
+<xacro:property name="props" value="${xacro.load_yaml(yaml_file)}"/>
+<xacro:property name="star" value="${props['/**']}"/>
+<xacro:property name="ros_parameters" value="${star['ros__parameters']}"/>
+<xacro:property name="wheel_radius" value="${ros_parameters['wheel_radius']}"/>
+<xacro:property name="track_width" value="${ros_parameters['track_width']}"/>
+<xacro:property name="collision_radius" value="${ros_parameters['collision_radius']}"/>
   <!-- Init colour -->
   <material name="black">
@@ -34,4 +40,8 @@
     <color rgba="1.0 1.0 1.0 1.0"/>
   </material>
+  <material name="purple">
+    <color rgba="0.3 0.16 0.52 1.0"/>
+  </material>
+  <xacro:arg name="color" default="purple"/>
   <link name="base_footprint"/>
   <joint name="base_joint" type="fixed">
@@ -46,10 +56,15 @@
         <mesh filename="package://nuturtle_description/meshes/burger_base.stl" scale="0.001 0.001 0.001"/>
       </geometry>
-      <material name="light_black"/>
+      <material name="$(arg color)"/>
     </visual>
     <collision>
       <origin xyz="-0.032 0 0.070" rpy="0 0 0"/>
       <geometry>
-        <box size="0.140 0.140 0.143"/>
+        <xacro:if value="${collision_radius &gt; 0.0}">
+          <cylinder radius="${collision_radius}" length="0.143"/>
+        </xacro:if>
+        <xacro:if value="${collision_radius &lt; 0.0}">
+          <box size="0.140 0.140 0.143"/>
+        </xacro:if>
       </geometry>
     </collision>
@@ -63,5 +78,5 @@
     <parent link="base_link"/>
     <child link="wheel_left_link"/>
-    <origin xyz="0.0 0.08 0.023" rpy="-1.57 0 0"/>
+    <origin xyz="0.0 ${0.5*track_width} 0.023" rpy="-1.57 0 0"/>
     <axis xyz="0 0 1"/>
   </joint>
@@ -77,5 +92,5 @@
       <origin xyz="0 0 0" rpy="0 0 0"/>
       <geometry>
-        <cylinder length="0.018" radius="0.033"/>
+        <cylinder length="0.018" radius="${wheel_radius}"/>
       </geometry>
     </collision>
@@ -89,5 +104,5 @@
     <parent link="base_link"/>
     <child link="wheel_right_link"/>
-    <origin xyz="0.0 -0.080 0.023" rpy="-1.57 0 0"/>
+    <origin xyz="0.0 ${-0.5*track_width} 0.023" rpy="-1.57 0 0"/>
     <axis xyz="0 0 1"/>
   </joint>
@@ -103,5 +118,5 @@
       <origin xyz="0 0 0" rpy="0 0 0"/>
       <geometry>
-        <cylinder length="0.018" radius="0.033"/>
+        <cylinder length="0.018" radius="${wheel_radius}"/>
       </geometry>
     </collision>
